Commit message: adjust finger2gsmini joint coordinate to be symmetrical

File: description/urdf/hand_gsmini.urdf (robot description, URDF)
Before this commit: robot hand, 5 links, 4 joints
Joints:
- joint finger_gsmini_joint_left: origin xyz=0 0.0120 0.0600 rpy=0 0 0 -> xyz=0 0.0120 0.0600 rpy=0 0 -1.570796327
- joint finger_gsmini_joint_right: origin xyz=0 -0.0120 0.0600 rpy=0 0 0 -> xyz=0 -0.0120 0.0600 rpy=0 0 1.570796327
