Commit message: add dummyLink/Joint for safe collision interaction

File: gsmini_panda_hand/urdf/hand_gsmini_tacto.urdf (robot description, URDF)
Before this commit: robot hand, 5 links, 4 joints
Links:
- added link dummylink; visual cylinder length=0.01 radius=0.005
- link panda_hand: mass 0.73 -> None
Joints:
- added joint dummyjoint: type prismatic, parent dummylink, child panda_hand, origin xyz=0 0 0 rpy=0 0 0, axis 0 1 0, limit lower=-0.0001 upper=0.0001 effort=100 velocity=0.001
- joint panda_finger_joint_left: limit lower=0.0 upper=0.04 effort=70 velocity=0.2 -> lower=0.0 upper=0.04 effort=100 velocity=0.2
- joint panda_finger_joint_right: limit lower=0.0 upper=0.04 effort=70 velocity=0.2 -> lower=0.0 upper=0.04 effort=100 velocity=0.2
